Commit message: Model improvements

File: models/thymio/model.urdf (robot description, URDF)
Before this commit: robot thymio, 4 links, 3 joints
Links:
- link caster: geometry collision cylinder length=.01 radius=.01; visual sphere radius=.01
Joints:
- removed joint caster_joint
- added joint z_caster_hinge: type continuous, parent chassis, child caster, origin xyz=0.043 0 -0.021 rpy=0 1.5707 1.5707, axis 0 0 1, limit lower=-2.8973 upper=2.8973 effort=0 velocity=7
